Commit message: Version 2.0

File: install/rover/share/rover/models/my_robot.urdf (robot description, URDF)
Before this commit: robot my_robot, 8 links, 7 joints
Joints:
- joint wheel_bl_joint: limit effort=20000 velocity=1.7 -> effort=2000 velocity=1.0
- joint wheel_br_joint: limit effort=20000 velocity=1.7 -> effort=2000 velocity=1.0
- joint wheel_fl_joint: limit effort=20000 velocity=1.7 -> effort=2000 velocity=1.0
- joint wheel_fr_joint: limit effort=20000 velocity=1.7 -> effort=2000 velocity=1.0

File: install/rover/share/rover/models/my_robot.urdf.xacro (robot description, xacro)
@@ -1,4 +1,4 @@
 <?xml version="1.0"?>
-<robot xmlns:xacro="http:/www.ros.org/wiki/xacro" name="my_robot">
+<robot xmlns:xacro="http:/www.ros.org/wiki/xacro" name="rover">
     <material name="grey">
         <color rgba="0.5 0.5 0.5 1"/>
@@ -31,14 +31,4 @@
         <child link="stand_link"/>
     </joint>
-    <!-- <joint name="camera_l_joint" type="fixed">
-        <origin xyz="${stand_length/2} ${stand_width/3} ${stand_height/2 - camera_height/2}"/>
-        <parent link="stand_link"/>
-        <child link="camera_l_link"/>
-    </joint>
-    <joint name="camera_r_joint" type="fixed">
-        <origin xyz="${stand_length/2} ${-stand_width/3} ${stand_height/2 - camera_height/2}"/>
-        <parent link="stand_link"/>
-        <child link="camera_r_link"/>
-    </joint> -->
     <joint name="lidar_joint" type="fixed">
         <origin xyz="0 0 ${stand_height/2 + camera_height/2}"/>
@@ -55,6 +45,5 @@
         <axis xyz="0 1 0"/>
         <origin xyz="${2*base_length/7} ${-base_width/2 - wheel_length/2} ${wheel_radius}" rpy="0 0 0"/>
-        <limit effort="20000" velocity="1.7"/>
-        <dynamics damping="1.0" friction="10.0"/>
+        <limit effort="2000" velocity="1.0"/>
     </joint>
     <joint name="wheel_fl_joint" type="continuous">
@@ -63,6 +52,5 @@
         <axis xyz="0 1 0"/>
         <origin xyz="${2*base_length/7} ${base_width/2 + wheel_length/2} ${wheel_radius}" rpy="0 0 0"/>
-        <limit effort="20000" velocity="1.7"/>
-        <dynamics damping="1.0" friction="10.0"/>
+        <limit effort="2000" velocity="1.0"/>
     </joint>
     <joint name="wheel_br_joint" type="continuous">
@@ -71,6 +59,5 @@
         <axis xyz="0 1 0"/>
         <origin xyz="${-2*base_length/7} ${-base_width/2 - wheel_length/2} ${wheel_radius}" rpy="0 0 0"/>
-        <limit effort="20000" velocity="1.7"/>
-        <dynamics damping="1.0" friction="10.0"/>
+        <limit effort="2000" velocity="1.0"/>
     </joint>
     <joint name="wheel_bl_joint" type="continuous">
@@ -79,6 +66,5 @@
         <axis xyz="0 1 0"/>
         <origin xyz="${-2*base_length/7} ${base_width/2 + wheel_length/2} ${wheel_radius}" rpy="0 0 0"/>
-        <limit effort="20000" velocity="1.7"/>
-        <dynamics damping="1.0" friction="10.0"/>
+        <limit effort="2000" velocity="1.0"/>
     </joint>
     <link name="base_link">
@@ -122,58 +108,4 @@
         </inertial>
     </link>
-    <!-- <link name="camera_l_link">
-        <visual>
-            <geometry>
-                <box size="${camera_length/2} ${camera_width} ${camera_height}"/>
-            </geometry>
-            <origin xyz="${-camera_length/4 + camera_length/2} 0 0" rpy="0 0 0"/>
-            <material name="white"/>
-        </visual>
-        <visual>
-            <geometry>
-                <cylinder radius="${camera_width/3.2}" length="${camera_length/2}"/>
-            </geometry>
-            <origin xyz="${camera_length/4 + camera_length/2} 0 0" rpy="0 ${pi/2} 0"/>
-            <material name="white"/>
-        </visual>
-        <collision>
-            <geometry>
-                <box size="${camera_length} ${camera_width} ${camera_height}"/>
-            </geometry>
-            <origin xyz="0 0 0" rpy="0 0 0"/>
-        </collision>
-        <inertial>
-            <origin xyz="0 0 0" rpy="0 0 0"/>
-            <mass value="${camera_mass}"/>
-            <inertia ixx="${(camera_mass/12)*(camera_height * camera_height + camera_length * camera_length)}" ixy="0" ixz="0" iyy="${(camera_mass/12)*(camera_height * camera_height + camera_width * camera_width)}" iyz="0" izz="${(camera_mass/12)*(camera_length * camera_length + camera_width * camera_width)}"/>
-        </inertial>
-    </link>
-    <link name="camera_r_link">
-        <visual>
-            <geometry>
-                <box size="${camera_length/2} ${camera_width} ${camera_height}"/>
-            </geometry>
-            <origin xyz="${-camera_length/4 + camera_length/2} 0 0" rpy="0 0 0"/>
-            <material name="white"/>
-        </visual>
-        <visual>
-            <geometry>
-                <cylinder radius="${camera_width/3.2}" length="${camera_length/2}"/>
-            </geometry>
-            <origin xyz="${camera_length/4 + camera_length/2} 0 0" rpy="0 ${pi/2} 0"/>
-            <material name="white"/>
-        </visual>
-        <collision>
-            <geometry>
-                <box size="${camera_length} ${camera_width} ${camera_height}"/>
-            </geometry>
-            <origin xyz="0 0 0" rpy="0 0 0"/>
-        </collision>
-        <inertial>
-            <origin xyz="0 0 0" rpy="0 0 0"/>
-            <mass value="${camera_mass}"/>
-            <inertia ixx="${(camera_mass/12)*(camera_height * camera_height + camera_length * camera_length)}" ixy="0" ixz="0" iyy="${(camera_mass/12)*(camera_height * camera_height + camera_width * camera_width)}" iyz="0" izz="${(camera_mass/12)*(camera_length * camera_length + camera_width * camera_width)}"/>
-        </inertial>
-    </link> -->
     <link name="lidar_link">
         <visual>

File: install/rover/share/rover/models/my_robot.xacro (robot description, xacro)
@@ -1,4 +1,4 @@
 <?xml version="1.0"?>
-<robot xmlns:xacro="http:/www.ros.org/wiki/xacro" name="my_robot">
+<robot xmlns:xacro="http:/www.ros.org/wiki/xacro" name="rover">
     <material name="grey">
         <color rgba="0.5 0.5 0.5 1"/>
@@ -10,4 +10,5 @@
         <color rgba="1 1 1 1"/>
     </material>
+    <!-- <xacro:property name="start_coord" value="30.2"/> -->
     <xacro:property name="base_length" value="1"/>
     <xacro:property name="base_width" value="0.6"/>
@@ -31,14 +32,4 @@
         <child link="stand_link"/>
     </joint>
-    <!-- <joint name="camera_l_joint" type="fixed">
-        <origin xyz="${stand_length/2} ${stand_width/3} ${stand_height/2 - camera_height/2}"/>
-        <parent link="stand_link"/>
-        <child link="camera_l_link"/>
-    </joint>
-    <joint name="camera_r_joint" type="fixed">
-        <origin xyz="${stand_length/2} ${-stand_width/3} ${stand_height/2 - camera_height/2}"/>
-        <parent link="stand_link"/>
-        <child link="camera_r_link"/>
-    </joint> -->
     <joint name="lidar_joint" type="fixed">
         <origin xyz="0 0 ${stand_height/2 + camera_height/4}"/>
@@ -51,6 +42,6 @@
         <axis xyz="0 1 0"/>
         <origin xyz="${2*base_length/7} ${-base_width/2 - wheel_length/2} ${wheel_radius}" rpy="0 0 0"/>
-        <limit effort="20000" velocity="1"/>
-        <dynamics damping="1.0" friction="1.0"/>
+        <limit effort="1000" velocity="0.75"/>
+        <!-- <dynamics damping="1.0" friction="1.0"/> -->
     </joint>
     <joint name="wheel_fl_joint" type="continuous">
@@ -59,6 +50,6 @@
         <axis xyz="0 1 0"/>
         <origin xyz="${2*base_length/7} ${base_width/2 + wheel_length/2} ${wheel_radius}" rpy="0 0 0"/>
-        <limit effort="20000" velocity="1"/>
-        <dynamics damping="1.0" friction="1.0"/>
+        <limit effort="1000" velocity="0.75"/>
+        <!-- <dynamics damping="1.0" friction="1.0"/> -->
     </joint>
     <joint name="wheel_br_joint" type="continuous">
@@ -67,6 +58,6 @@
         <axis xyz="0 1 0"/>
         <origin xyz="${-2*base_length/7} ${-base_width/2 - wheel_length/2} ${wheel_radius}" rpy="0 0 0"/>
-        <limit effort="20000" velocity="1"/>
-        <dynamics damping="1.0" friction="1.0"/>
+        <limit effort="1000" velocity="0.75"/>
+        <!-- <dynamics damping="1.0" friction="1.0"/> -->
     </joint>
     <joint name="wheel_bl_joint" type="continuous">
@@ -75,6 +66,6 @@
         <axis xyz="0 1 0"/>
         <origin xyz="${-2*base_length/7} ${base_width/2 + wheel_length/2} ${wheel_radius}" rpy="0 0 0"/>
-        <limit effort="20000" velocity="1"/>
-        <dynamics damping="1.0" friction="1.0"/>
+        <limit effort="1000" velocity="0.75"/>
+        <!-- <dynamics damping="1.0" friction="1.0"/> -->
     </joint>
     <link name="base_link">
@@ -97,10 +88,4 @@
             <inertia ixx="${(base_mass/12)*(base_height * base_height + base_length * base_length)}" ixy="0" ixz="0" iyy="${(base_mass/12)*(base_height * base_height + base_width * base_width)}" iyz="0" izz="${(base_mass/12)*(base_length * base_length + base_width * base_width)}"/>
         </inertial>
-        <sensor name="imu_sensor" type="imu">
-            <always_on>1</always_on>
-            <update_rate>2</update_rate>
-            <visualize>true</visualize>
-            <topic>imu</topic>
-        </sensor>
     </link>
     <link name="stand_link">
@@ -124,59 +109,4 @@
         </inertial>
     </link>
-<!--
-    <link name="camera_l_link">
-        <visual>
-            <geometry>
-                <box size="${camera_length/2} ${camera_width} ${camera_height}"/>
-            </geometry>
-            <origin xyz="${-camera_length/4 + camera_length/2} 0 0" rpy="0 0 0"/>
-            <material name="white"/>
-        </visual>
-        <visual>
-            <geometry>
-                <cylinder radius="${camera_width/3.2}" length="${camera_length/2}"/>
-            </geometry>
-            <origin xyz="${camera_length/4 + camera_length/2} 0 0" rpy="0 ${pi/2} 0"/>
-            <material name="white"/>
-        </visual>
-        <collision>
-            <geometry>
-                <box size="${camera_length} ${camera_width} ${camera_height}"/>
-            </geometry>
-            <origin xyz="0 0 0" rpy="0 0 0"/>
-        </collision>
-        <inertial>
-            <origin xyz="0 0 0" rpy="0 0 0"/>
-            <mass value="${camera_mass}"/>
-            <inertia ixx="${(camera_mass/12)*(camera_height * camera_height + camera_length * camera_length)}" ixy="0" ixz="0" iyy="${(camera_mass/12)*(camera_height * camera_height + camera_width * camera_width)}" iyz="0" izz="${(camera_mass/12)*(camera_length * camera_length + camera_width * camera_width)}"/>
-        </inertial>
-    </link>
-    <link name="camera_r_link">
-        <visual>
-            <geometry>
-                <box size="${camera_length/2} ${camera_width} ${camera_height}"/>
-            </geometry>
-            <origin xyz="${-camera_length/4 + camera_length/2} 0 0" rpy="0 0 0"/>
-            <material name="white"/>
-        </visual>
-        <visual>
-            <geometry>
-                <cylinder radius="${camera_width/3.2}" length="${camera_length/2}"/>
-            </geometry>
-            <origin xyz="${camera_length/4 + camera_length/2} 0 0" rpy="0 ${pi/2} 0"/>
-            <material name="white"/>
-        </visual>
-        <collision>
-            <geometry>
-                <box size="${camera_length} ${camera_width} ${camera_height}"/>
-            </geometry>
-            <origin xyz="0 0 0" rpy="0 0 0"/>
-        </collision>
-        <inertial>
-            <origin xyz="0 0 0" rpy="0 0 0"/>
-            <mass value="${camera_mass}"/>
-            <inertia ixx="${(camera_mass/12)*(camera_height * camera_height + camera_length * camera_length)}" ixy="0" ixz="0" iyy="${(camera_mass/12)*(camera_height * camera_height + camera_width * camera_width)}" iyz="0" izz="${(camera_mass/12)*(camera_length * camera_length + camera_width * camera_width)}"/>
-        </inertial>
-    </link> -->
     <link name="lidar_link">
         <visual>
@@ -198,32 +128,4 @@
             <inertia ixx="${(camera_mass/12)*(3 * camera_width/2 * camera_width/2 + camera_length/2 * camera_length/2)}" ixy="0" ixz="0" iyy="${(camera_mass/12)*(3 * camera_width/2 * camera_width/2 + camera_length/2 * camera_length/2)}" iyz="0" izz="${(camera_mass * camera_width/2 * camera_width/2) / 2}"/>
         </inertial>
-        <sensor name='gpu_lidar' type='gpu_lidar'>"
-            <pose relative_to='lidar_frame'>0 0 0 0 0 0</pose>
-            <topic>lidar</topic>
-            <update_rate>1</update_rate>
-            <ray>
-                <scan>
-                    <horizontal>
-                        <samples>2800</samples>
-                        <resolution>1</resolution>
-                        <min_angle>${-pi}</min_angle>
-                        <max_angle>${pi}</max_angle>
-                    </horizontal>
-                    <vertical>
-                        <samples>640</samples>
-                        <resolution>1</resolution>
-                        <min_angle>${-pi/4}</min_angle>
-                        <max_angle>${-pi/16}</max_angle>
-                    </vertical>
-                </scan>
-                <range>
-                    <min>0.08</min>
-                    <max>10.0</max>
-                    <resolution>0.01</resolution>
-                </range>
-            </ray>
-            <always_on>1</always_on>
-            <visualize>true</visualize>
-        </sensor>
     </link>
     <link name="wheel_fr_link">
